Commit message: Created simulated lidar and added it to the robot description. Added a launch file to launch the simulation with Gazebo and the robot.

File: description/robot.urdf.xacro (robot description, xacro)
@@ -3,3 +3,5 @@
     <!-- Example link -->
     <xacro:include filename="robot_core.xacro" />
+    <xacro:include filename="gazebo_control.xacro" />
+    <xacro:include filename="lidar.xacro"/>
 </robot>

File: description/robot_core.xacro (robot description, xacro)
@@ -13,4 +13,7 @@
     <material name = "black">
         <color rgba = "0 0 0 1"/>
+    </material>
+    <material name = "red">
+        <color rgba = "1 0 0 1"/>
     </material>
     <!-- Base link  -->
@@ -109,3 +112,7 @@
         </xacro:inertial_sphere>
     </link>
+    <gazebo reference="caster_wheel">
+        <mu1>0.001</mu1>
+        <mu2>0.001</mu2>
+    </gazebo>
 </robot>
